Commit message: improve model and include safety flange sphere
.. as documented in the support forum.

File: cu_ur5e_description/urdf/mounted_arm.urdf.xacro (robot description, xacro)
@@ -8,4 +8,7 @@
         safety_limits="true"
         />
+    <material name="mount_gray">
+                <color rgba="0.4 0.4 0.4 1"/>
+    </material>
     <xacro:property name="mount_height" value="0.8"/>
     <link name="mount">
@@ -15,7 +18,5 @@
             </geometry>
             <origin xyz="0 0 ${mount_height / 2}" rpy="0 0 0"/>
-            <material name="gray">
-                <color rgba="0.5 0.5 0.5 1"/>
-            </material>
+            <material name="mount_gray" />
         </visual>
         <visual>
@@ -24,7 +25,5 @@
             </geometry>
             <origin xyz="0 0 ${mount_height - 0.0065}" rpy="0 0 0"/>
-            <material name="gray">
-                <color rgba="0.5 0.5 0.5 1"/>
-            </material>
+            <material name="mount_gray" />
         </visual>
         <visual>
@@ -33,7 +32,5 @@
             </geometry>
             <origin xyz="0 0 ${0 + 0.025}" rpy="0 0 ${tau/4}"/>
-            <material name="gray">
-                <color rgba="0.5 0.5 0.5 1"/>
-            </material>
+            <material name="mount_gray" />
         </visual>
         <visual>
@@ -42,7 +39,5 @@
             </geometry>
             <origin xyz="0 0 ${0 + 0.025}" rpy="0 0 ${tau/4+tau/6}"/>
-            <material name="gray">
-                <color rgba="0.5 0.5 0.5 1"/>
-            </material>
+            <material name="mount_gray" />
         </visual>
         <visual>
@@ -51,7 +46,5 @@
             </geometry>
             <origin xyz="0 0 ${0 + 0.025}" rpy="0 0 ${tau/4-tau/6}"/>
-            <material name="gray">
-                <color rgba="0.5 0.5 0.5 1"/>
-            </material>
+            <material name="mount_gray" />
         </visual>
         <collision>
@@ -79,7 +72,5 @@
             </geometry>
             <origin xyz="0.0 0 0.0" rpy="0 0 0"/>
-            <material name="gray">
-                <color rgba="0.5 0.5 0.5 1"/>
-            </material>
+            <material name="LightGrey" />
         </visual>
         <collision>
@@ -95,25 +86,26 @@
         <origin xyz="-0.3 0.0 0.5" rpy="0 0 0"/>
     </joint>
-    <link name="wall">
+    <link name="arm_flange_safety">
+        <!-- https://forum.universal-robots.com/t/error-c403a0-danger-of-clamping-between-the-robot-lower-arm-and-tool/16142/2 -->
         <visual>
             <geometry>
-                <box size="0.1 4.0 2.0"/>
+                <sphere radius="0"/>
             </geometry>
-            <origin xyz="0 0 1.0" rpy="0 0 0"/>
-            <material name="gray">
-                <color rgba="0.5 0.5 0.5 1"/>
+            <origin xyz="0 0 0.0" rpy="0 0 0"/>
+            <material name="transparent_gray">
+                <color rgba="0.5 0.5 0.5 .3"/>
             </material>
         </visual>
         <collision>
             <geometry>
-                <box size="0.1 4.0 2.0"/>
+                <sphere radius="${0.0375+0.028}"/>
             </geometry>
-            <origin xyz="0 0 1.0" rpy="0 0 0"/>
+            <origin xyz="0 0 0.0" rpy="0 0 0"/>
         </collision>
     </link>
-    <joint name="base_to_wall" type="fixed">
-        <parent link="base"/>
-        <child link="wall"/>
-        <origin xyz="-.5 0 0" rpy="0 0 0"/>
+    <joint name="arm_flange_safety_joint" type="fixed">
+        <parent link="arm_flange"/>
+        <child link="arm_flange_safety"/>
+        <origin xyz="0 0 0.0" rpy="0 0 0"/>
     </joint>
 </robot>

Commit message: add tool change adapter to urdf
(only tested in student workspace)

File: cu_ur5e_description/urdf/mounted_arm.urdf.xacro (robot description, xacro)
@@ -86,4 +86,26 @@
         <origin xyz="-0.3 0.0 0.5" rpy="0 0 0"/>
     </joint> -->
+    <xacro:property name="adapter_len" value="0.022"/>   <!-- 4 cm -->
+    <xacro:property name="adapter_rad" value="0.035"/>  <!-- 3.5 cm -->
+    <link name="arm_ee_adapter">
+    <visual>
+        <origin xyz="0 0 ${adapter_len/2}" rpy="0 0 0"/>
+        <geometry>
+        <cylinder length="${adapter_len}" radius="${adapter_rad}"/>
+        </geometry>
+        <material name="mount_gray"/>
+    </visual>
+    <collision>
+        <origin xyz="0 0 ${adapter_len/2}" rpy="0 0 0"/>
+        <geometry>
+        <cylinder length="${adapter_len}" radius="${adapter_rad}"/>
+        </geometry>
+    </collision>
+    </link>
+    <joint name="arm_flange_to_adapter" type="fixed">
+    <parent link="arm_tool0"/>
+    <child link="arm_ee_adapter"/>
+    <origin xyz="0 0 0" rpy="0 0 0"/>
+    </joint>
     <link name="arm_flange_safety">
         <!-- https://forum.universal-robots.com/t/error-c403a0-danger-of-clamping-between-the-robot-lower-arm-and-tool/16142/2 -->
