Commit message: move operator table
rearranging room logistics (likely not the last time)

File: cu_ur5e_description/robots/basic_setup.urdf.xacro (robot description, xacro)
@@ -39,5 +39,5 @@
         <parent link="base"/>
         <child link="operator_table"/>
-        <origin xyz="0.0 ${-0.8-.65} 0.0" rpy="0 0 0"/>
+        <origin xyz="0.0 ${0.8+.65} 0.0" rpy="0 0 0"/>
     </joint>
     <xacro:property name="clearance_height" value="0.55"/>

Commit message: rearranged robot setup with moveit config

File: cu_ur5e_description/robots/basic_setup.urdf.xacro (robot description, xacro)
@@ -29,9 +29,9 @@
         <origin xyz="-.5 0 0" rpy="0 0 0"/>
     </joint>
-    <xacro:table length="0.8" width="0.8" height="0.72" name="table" />
+    <xacro:table length="0.6" width="1." height="0.74" name="table" />
     <joint name="base_to_table" type="fixed">
         <parent link="base"/>
         <child link="table"/>
-        <origin xyz="0.85 0 0.0" rpy="0 0 0"/>
+        <origin xyz="${0.3+0.45} -0.11 0.0" rpy="0 0 0"/>
     </joint>
     <xacro:table length="0.8" width="1.6" height="0.72" name="operator_table" />
@@ -39,5 +39,5 @@
         <parent link="base"/>
         <child link="operator_table"/>
-        <origin xyz="0.0 ${0.8+.65} 0.0" rpy="0 0 0"/>
+        <origin xyz="0.0 ${-0.8-.75} 0.0" rpy="0 0 0"/>
     </joint>
     <xacro:property name="clearance_height" value="0.55"/>
@@ -56,3 +56,9 @@
         <origin xyz="0.0 0.0 ${clearance_height/2}" rpy="0 0 0"/>
     </joint>
+    <xacro:table length="0.8" width="0.8" height="0.72" name="side_table" />
+    <joint name="base_to_side_table" type="fixed">
+        <parent link="base"/>
+        <child link="side_table"/>
+        <origin xyz="0.0 ${0.4+0.45} 0.0" rpy="0 0 0"/>
+    </joint>
 </robot>

File: cu_ur5e_description/urdf/mounted_arm.urdf.xacro (robot description, xacro)
@@ -64,5 +64,5 @@
         <parent link="base"/>
         <child link="mount"/>
-        <origin xyz="0 0 0.0" rpy="0 0 0"/>
+        <origin xyz="0 0 0.0" rpy="0 0 ${tau/4}"/>
     </joint>
     <link name="control_box">

File: cu_ur5e_description/urdf/table.urdf.xacro (robot description, xacro)
@@ -59,5 +59,5 @@
         <parent link="${name}"/>
         <child link="${name}_top"/>
-        <origin xyz="0 0 0.72" rpy="0 0 0"/>
+        <origin xyz="0 0 ${height}" rpy="0 0 0"/>
     </joint>
 </xacro:macro>

Commit message: move table closer

File: cu_ur5e_description/robots/basic_setup.urdf.xacro (robot description, xacro)
@@ -33,5 +33,5 @@
         <parent link="base"/>
         <child link="table"/>
-        <origin xyz="${0.3+0.45} -0.11 0.0" rpy="0 0 0"/>
+        <origin xyz="${0.3+0.33} -0.11 0.0" rpy="0 0 0"/>
     </joint>
     <xacro:table length="0.8" width="1.6" height="0.72" name="operator_table" />

Commit message: update geometry

File: cu_ur5e_description/robots/basic_setup.urdf.xacro (robot description, xacro)
@@ -29,9 +29,9 @@
         <origin xyz="-.5 0 0" rpy="0 0 0"/>
     </joint>
-    <xacro:table length="0.6" width="1." height="0.74" name="table" />
+    <xacro:table length="0.8" width="0.8" height="0.72" name="table" />
     <joint name="base_to_table" type="fixed">
         <parent link="base"/>
         <child link="table"/>
-        <origin xyz="${0.3+0.33} -0.11 0.0" rpy="0 0 0"/>
+        <origin xyz="${0.4+0.33} -0.11 0.0" rpy="0 0 0"/>
     </joint>
     <xacro:table length="0.8" width="1.6" height="0.72" name="operator_table" />
@@ -62,3 +62,24 @@
         <origin xyz="0.0 ${0.4+0.45} 0.0" rpy="0 0 0"/>
     </joint>
+    <xacro:property name="tripod_height" value="1.45"/>
+    <link name="tripod">
+        <visual>
+            <geometry>
+                <cylinder length="${tripod_height}" radius="0.15"/>
+                <origin xyz="0 0 0" rpy="0 0 0"/>
+            </geometry>
+            <material name="mount_gray" />
+        </visual>
+        <collision>
+            <geometry>
+                <cylinder length="${tripod_height}" radius="0.15"/>
+            </geometry>
+            <origin xyz="0 0 0" rpy="0 0 0"/>
+        </collision>
+    </link>
+    <joint name="base_to_tripod" type="fixed">
+        <parent link="base"/>
+        <child link="tripod"/>
+        <origin xyz="-0.4 -0.5 ${tripod_height/2}" rpy="0 0 0"/>
+    </joint>
 </robot>

File: cu_ur5e_description/urdf/mounted_arm.urdf.xacro (robot description, xacro)
@@ -66,5 +66,5 @@
         <origin xyz="0 0 0.0" rpy="0 0 ${tau/4}"/>
     </joint>
-    <link name="control_box">
+    <!-- <link name="control_box">
         <visual>
             <geometry>
@@ -85,5 +85,5 @@
         <child link="control_box"/>
         <origin xyz="-0.3 0.0 0.5" rpy="0 0 0"/>
-    </joint>
+    </joint> -->
     <link name="arm_flange_safety">
         <!-- https://forum.universal-robots.com/t/error-c403a0-danger-of-clamping-between-the-robot-lower-arm-and-tool/16142/2 -->

Commit message: add missing collision geometry to clearance

File: cu_ur5e_description/robots/basic_setup.urdf.xacro (robot description, xacro)
@@ -50,4 +50,10 @@
             <material name="clearance_volume"/>
         </visual>
+        <collision>
+            <geometry>
+                <box size="0.8 1.6 ${clearance_height}"/>
+            </geometry>
+            <origin xyz="0 0 0.0" rpy="0 0 0"/>
+        </collision>
     </link>
     <joint name="operator_clearance_joint" type="fixed">

Commit message: update environment to changed tables

File: cu_ur5e_description/robots/basic_setup.urdf.xacro (robot description, xacro)
@@ -9,4 +9,24 @@
         <color rgba="0.6 0.4 0.2 0.2"/>
     </material>
+    <link name="wall_indent">
+        <visual>
+            <geometry>
+                <box size="0.18 0.74 2.0"/>
+            </geometry>
+            <origin xyz="0 0 0" rpy="0 0 0"/>
+            <material name="wall_gray"/>
+        </visual>
+        <collision>
+            <geometry>
+                <box size="0.18 0.74 2.0"/>
+            </geometry>
+            <origin xyz="0 0 0" rpy="0 0 0"/>
+        </collision>
+    </link>
+    <joint name="base_to_wall_indent" type="fixed">
+        <parent link="base"/>
+        <child link="wall_indent"/>
+        <origin xyz="-0.60 0.1 1" rpy="0 0 0"/>
+    </joint>
     <link name="wall">
         <visual>
@@ -14,5 +34,5 @@
                 <box size="0.1 4.5 2.0"/>
             </geometry>
-            <origin xyz="0 0 1.0" rpy="0 0 0"/>
+            <origin xyz="-0.235 0 1.0" rpy="0 0 0"/>
             <material name="wall_gray"/>
         </visual>
@@ -21,5 +41,5 @@
                 <box size="0.1 4.0 2.0"/>
             </geometry>
-            <origin xyz="0 0 1.0" rpy="0 0 0"/>
+            <origin xyz="-0.235 0 1.0" rpy="0 0 0"/>
         </collision>
     </link>
@@ -29,9 +49,9 @@
         <origin xyz="-.5 0 0" rpy="0 0 0"/>
     </joint>
-    <xacro:table length="0.8" width="0.8" height="0.72" name="table" />
+    <xacro:table length="0.8" width="1.6" height="0.72" name="table" />
     <joint name="base_to_table" type="fixed">
         <parent link="base"/>
         <child link="table"/>
-        <origin xyz="${0.4+0.33} -0.11 0.0" rpy="0 0 0"/>
+        <origin xyz="${0.4+0.11} -0.11 0.0" rpy="0 0 0"/>
     </joint>
     <xacro:table length="0.8" width="1.6" height="0.72" name="operator_table" />
@@ -39,5 +59,5 @@
         <parent link="base"/>
         <child link="operator_table"/>
-        <origin xyz="0.0 ${-0.8-.75} 0.0" rpy="0 0 0"/>
+        <origin xyz="-0.29 ${-0.8-.75} 0.0" rpy="0 0 0"/>
     </joint>
     <xacro:property name="clearance_height" value="0.55"/>
@@ -66,5 +86,5 @@
         <parent link="base"/>
         <child link="side_table"/>
-        <origin xyz="0.0 ${0.4+0.45} 0.0" rpy="0 0 0"/>
+        <origin xyz="-0.29 ${0.4+0.45} 0.0" rpy="0 0 0"/>
     </joint>
     <xacro:property name="tripod_height" value="1.45"/>
